File: hw-design/peripherals.sch (KiCad schematic (older format))
At the start: 36 parts, among them P8 CONN_01X17, P9 CONN_01X17, Q2 BC847, Q3 BC847, Q4 BC847, Q5 BC847, Q6 BC847, Q7 BC847, U10 China-0038, U11 China-0038, U12 China-0038, U13 China-0038

Commit message: Changed to 2 boards layout. On the top one there is only : speaker, IR stuff, RGB led.
Connections:
- net +3V3 renamed +3.3VP
- net +5V: no longer names the net of P9.13 (P13)
- net +BATT renamed VAA
- net GND renamed GNDA
- no-connect marks 23 -> 24

Commit message: Another idea of PCB split.
Parts:
- P8, P9: footprint w_pin_strip:pin_strip_17 -> iwasz:pin_socket_17
Changed lines of the file:
@@
 $Descr A4 11693 8268
 encoding utf-8
-Sheet 6 6
+Sheet 6 7
 Title ""
 Date ""
@@
 F 0 "P8" H 6025 2875 50  0000 L CNN
 F 1 "CONN_01X17" H 6025 2975 50  0000 L CNN
-F 2 "w_pin_strip:pin_strip_17" H 6325 3900 50  0001 C CNN
+F 2 "iwasz:pin_socket_17" H 6325 3900 50  0001 C CNN
 F 3 "" H 6325 3900 50  0000 C CNN
 	1    6325 3900
@@
 F 0 "P9" H 6175 2875 50  0000 L CNN
 F 1 "CONN_01X17" H 6175 2975 50  0000 L CNN
-F 2 "w_pin_strip:pin_strip_17" H 6475 3900 50  0001 C CNN
+F 2 "iwasz:pin_socket_17" H 6475 3900 50  0001 C CNN
 F 3 "" H 6475 3900 50  0000 C CNN
 	1    6475 3900
@@
 sound
 $Comp
-L GNDA #PWR72
+L GNDA #PWR65
 U 1 1 58175484
 P 5550 4600
-F 0 "#PWR72" H 5550 4350 50  0001 C CNN
+F 0 "#PWR65" H 5550 4350 50  0001 C CNN
 F 1 "GNDA" V 5555 4473 50  0000 R CNN
 F 2 "" H 5550 4600 50  0000 C CNN
@@
 $EndComp
 $Comp
-L GNDA #PWR74
+L GNDA #PWR67
 U 1 1 58176096
 P 6975 4200
-F 0 "#PWR74" H 6975 3950 50  0001 C CNN
+F 0 "#PWR67" H 6975 3950 50  0001 C CNN
 F 1 "GNDA" V 6980 4072 50  0000 R CNN
 F 2 "" H 6975 4200 50  0000 C CNN
@@
 $EndComp
 $Comp
-L GNDA #PWR78
+L GNDA #PWR71
 U 1 1 58176881
 P 10275 6125
-F 0 "#PWR78" H 10275 5875 50  0001 C CNN
+F 0 "#PWR71" H 10275 5875 50  0001 C CNN
 F 1 "GNDA" H 10280 5952 50  0000 C CNN
 F 2 "" H 10275 6125 50  0000 C CNN
@@
 $EndComp
 $Comp
-L GNDA #PWR69
+L GNDA #PWR62
 U 1 1 58177DAF
 P 3600 6975
-F 0 "#PWR69" H 3600 6725 50  0001 C CNN
+F 0 "#PWR62" H 3600 6725 50  0001 C CNN
 F 1 "GNDA" H 3605 6802 50  0000 C CNN
 F 2 "" H 3600 6975 50  0000 C CNN
@@
 $EndComp
 $Comp
-L GNDA #PWR64
+L GNDA #PWR57
 U 1 1 58177F9A
 P 2300 6975
-F 0 "#PWR64" H 2300 6725 50  0001 C CNN
+F 0 "#PWR57" H 2300 6725 50  0001 C CNN
 F 1 "GNDA" H 2305 6802 50  0000 C CNN
 F 2 "" H 2300 6975 50  0000 C CNN
@@
 $EndComp
 $Comp
-L GNDA #PWR76
+L GNDA #PWR69
 U 1 1 58178DD9
 P 9550 2325
-F 0 "#PWR76" H 9550 2075 50  0001 C CNN
+F 0 "#PWR69" H 9550 2075 50  0001 C CNN
 F 1 "GNDA" H 9555 2152 50  0000 C CNN
 F 2 "" H 9550 2325 50  0000 C CNN
@@
 $EndComp
 $Comp
-L GNDA #PWR70
+L GNDA #PWR63
 U 1 1 581793B3
 P 3625 2100
-F 0 "#PWR70" H 3625 1850 50  0001 C CNN
+F 0 "#PWR63" H 3625 1850 50  0001 C CNN
 F 1 "GNDA" H 3630 1927 50  0000 C CNN
 F 2 "" H 3625 2100 50  0000 C CNN
@@
 $EndComp
 $Comp
-L GNDA #PWR66
+L GNDA #PWR59
 U 1 1 5817A170
 P 2850 2100
-F 0 "#PWR66" H 2850 1850 50  0001 C CNN
+F 0 "#PWR59" H 2850 1850 50  0001 C CNN
 F 1 "GNDA" H 2855 1927 50  0000 C CNN
 F 2 "" H 2850 2100 50  0000 C CNN
@@
 $EndComp
 $Comp
-L GNDA #PWR62
+L GNDA #PWR55
 U 1 1 5817A1E7
 P 2075 2100
-F 0 "#PWR62" H 2075 1850 50  0001 C CNN
+F 0 "#PWR55" H 2075 1850 50  0001 C CNN
 F 1 "GNDA" H 2080 1927 50  0000 C CNN
 F 2 "" H 2075 2100 50  0000 C CNN
@@
 $EndComp
 $Comp
-L GNDA #PWR60
+L GNDA #PWR53
 U 1 1 5817A25E
 P 1300 2100
-F 0 "#PWR60" H 1300 1850 50  0001 C CNN
+F 0 "#PWR53" H 1300 1850 50  0001 C CNN
 F 1 "GNDA" H 1305 1927 50  0000 C CNN
 F 2 "" H 1300 2100 50  0000 C CNN
@@
 NoConn ~ 6750 3500
 $Comp
-L +3.3VP #PWR71
+L +3.3VP #PWR64
 U 1 1 5817DDD0
 P 5550 4400
-F 0 "#PWR71" H 5700 4350 50  0001 C CNN
+F 0 "#PWR64" H 5700 4350 50  0001 C CNN
 F 1 "+3.3VP" V 5570 4498 50  0000 L CNN
 F 2 "" H 5550 4400 50  0000 C CNN
@@
 $EndComp
 $Comp
-L +3.3VP #PWR68
+L +3.3VP #PWR61
 U 1 1 5817DF9D
 P 3600 5500
-F 0 "#PWR68" H 3750 5450 50  0001 C CNN
+F 0 "#PWR61" H 3750 5450 50  0001 C CNN
 F 1 "+3.3VP" H 3620 5643 50  0000 C CNN
 F 2 "" H 3600 5500 50  0000 C CNN
@@
 $EndComp
 $Comp
-L +3.3VP #PWR63
+L +3.3VP #PWR56
 U 1 1 5817E8B4
 P 2300 5500
-F 0 "#PWR63" H 2450 5450 50  0001 C CNN
+F 0 "#PWR56" H 2450 5450 50  0001 C CNN
 F 1 "+3.3VP" H 2320 5643 50  0000 C CNN
 F 2 "" H 2300 5500 50  0000 C CNN
@@
 $EndComp
 $Comp
-L +3.3VP #PWR77
+L +3.3VP #PWR70
 U 1 1 5817F6CE
 P 10075 3975
-F 0 "#PWR77" H 10225 3925 50  0001 C CNN
+F 0 "#PWR70" H 10225 3925 50  0001 C CNN
 F 1 "+3.3VP" H 10095 4118 50  0000 C CNN
 F 2 "" H 10075 3975 50  0000 C CNN
@@
 $EndComp
 $Comp
-L +3.3VP #PWR59
+L +3.3VP #PWR52
 U 1 1 581811E3
 P 875 2475
-F 0 "#PWR59" H 1025 2425 50  0001 C CNN
+F 0 "#PWR52" H 1025 2425 50  0001 C CNN
 F 1 "+3.3VP" H 895 2618 50  0000 C CNN
 F 2 "" H 875 2475 50  0000 C CNN
@@
 $EndComp
 $Comp
-L +3.3VP #PWR61
+L +3.3VP #PWR54
 U 1 1 58182A98
 P 1650 2475
-F 0 "#PWR61" H 1800 2425 50  0001 C CNN
+F 0 "#PWR54" H 1800 2425 50  0001 C CNN
 F 1 "+3.3VP" H 1670 2618 50  0000 C CNN
 F 2 "" H 1650 2475 50  0000 C CNN
@@
 $EndComp
 $Comp
-L +3.3VP #PWR65
+L +3.3VP #PWR58
 U 1 1 58182C81
 P 2425 2475
-F 0 "#PWR65" H 2575 2425 50  0001 C CNN
+F 0 "#PWR58" H 2575 2425 50  0001 C CNN
 F 1 "+3.3VP" H 2445 2618 50  0000 C CNN
 F 2 "" H 2425 2475 50  0000 C CNN
@@
 $EndComp
 $Comp
-L +3.3VP #PWR67
+L +3.3VP #PWR60
 U 1 1 58183424
 P 3200 2475
-F 0 "#PWR67" H 3350 2425 50  0001 C CNN
+F 0 "#PWR60" H 3350 2425 50  0001 C CNN
 F 1 "+3.3VP" H 3220 2618 50  0000 C CNN
 F 2 "" H 3200 2475 50  0000 C CNN
@@
 $EndComp
 $Comp
-L VAA #PWR73
+L VAA #PWR66
 U 1 1 58184D5C
 P 6025 3500
-F 0 "#PWR73" H 6025 3350 50  0001 C CNN
+F 0 "#PWR66" H 6025 3350 50  0001 C CNN
 F 1 "VAA" V 6043 3627 50  0000 L CNN
 F 2 "" H 6025 3500 50  0000 C CNN
@@
 $EndComp
 $Comp
-L VAA #PWR75
+L VAA #PWR68
 U 1 1 58185AC0
 P 9550 1400
-F 0 "#PWR75" H 9550 1250 50  0001 C CNN
+F 0 "#PWR68" H 9550 1250 50  0001 C CNN
 F 1 "VAA" H 9567 1573 50  0000 C CNN
 F 2 "" H 9550 1400 50  0000 C CNN

Commit message: 2 boards and 1 little with color sensors.
Connections:
- net VAA: now also P8.13 (P13); no longer P8.5 (P5)
Changed lines of the file:
@@
 Wire Wire Line
 	6675 3500 6750 3500
-Wire Wire Line
-	6025 3500 6125 3500
 NoConn ~ 6125 4500
-NoConn ~ 6125 4300
 NoConn ~ 6125 4200
 NoConn ~ 6125 4100
@@
 sound
 $Comp
-L GNDA #PWR65
+L GNDA #PWR052
 U 1 1 58175484
 P 5550 4600
-F 0 "#PWR65" H 5550 4350 50  0001 C CNN
+F 0 "#PWR052" H 5550 4350 50  0001 C CNN
 F 1 "GNDA" V 5555 4473 50  0000 R CNN
 F 2 "" H 5550 4600 50  0000 C CNN
@@
 $EndComp
 $Comp
-L GNDA #PWR67
+L GNDA #PWR053
 U 1 1 58176096
 P 6975 4200
-F 0 "#PWR67" H 6975 3950 50  0001 C CNN
+F 0 "#PWR053" H 6975 3950 50  0001 C CNN
 F 1 "GNDA" V 6980 4072 50  0000 R CNN
 F 2 "" H 6975 4200 50  0000 C CNN
@@
 $EndComp
 $Comp
-L GNDA #PWR71
+L GNDA #PWR054
 U 1 1 58176881
 P 10275 6125
-F 0 "#PWR71" H 10275 5875 50  0001 C CNN
+F 0 "#PWR054" H 10275 5875 50  0001 C CNN
 F 1 "GNDA" H 10280 5952 50  0000 C CNN
 F 2 "" H 10275 6125 50  0000 C CNN
@@
 $EndComp
 $Comp
-L GNDA #PWR62
+L GNDA #PWR055
 U 1 1 58177DAF
 P 3600 6975
-F 0 "#PWR62" H 3600 6725 50  0001 C CNN
+F 0 "#PWR055" H 3600 6725 50  0001 C CNN
 F 1 "GNDA" H 3605 6802 50  0000 C CNN
 F 2 "" H 3600 6975 50  0000 C CNN
@@
 $EndComp
 $Comp
-L GNDA #PWR57
+L GNDA #PWR056
 U 1 1 58177F9A
 P 2300 6975
-F 0 "#PWR57" H 2300 6725 50  0001 C CNN
+F 0 "#PWR056" H 2300 6725 50  0001 C CNN
 F 1 "GNDA" H 2305 6802 50  0000 C CNN
 F 2 "" H 2300 6975 50  0000 C CNN
@@
 $EndComp
 $Comp
-L GNDA #PWR69
+L GNDA #PWR057
 U 1 1 58178DD9
 P 9550 2325
-F 0 "#PWR69" H 9550 2075 50  0001 C CNN
+F 0 "#PWR057" H 9550 2075 50  0001 C CNN
 F 1 "GNDA" H 9555 2152 50  0000 C CNN
 F 2 "" H 9550 2325 50  0000 C CNN
@@
 $EndComp
 $Comp
-L GNDA #PWR63
+L GNDA #PWR058
 U 1 1 581793B3
 P 3625 2100
-F 0 "#PWR63" H 3625 1850 50  0001 C CNN
+F 0 "#PWR058" H 3625 1850 50  0001 C CNN
 F 1 "GNDA" H 3630 1927 50  0000 C CNN
 F 2 "" H 3625 2100 50  0000 C CNN
@@
 $EndComp
 $Comp
-L GNDA #PWR59
+L GNDA #PWR059
 U 1 1 5817A170
 P 2850 2100
-F 0 "#PWR59" H 2850 1850 50  0001 C CNN
+F 0 "#PWR059" H 2850 1850 50  0001 C CNN
 F 1 "GNDA" H 2855 1927 50  0000 C CNN
 F 2 "" H 2850 2100 50  0000 C CNN
@@
 $EndComp
 $Comp
-L GNDA #PWR55
+L GNDA #PWR060
 U 1 1 5817A1E7
 P 2075 2100
-F 0 "#PWR55" H 2075 1850 50  0001 C CNN
+F 0 "#PWR060" H 2075 1850 50  0001 C CNN
 F 1 "GNDA" H 2080 1927 50  0000 C CNN
 F 2 "" H 2075 2100 50  0000 C CNN
@@
 $EndComp
 $Comp
-L GNDA #PWR53
+L GNDA #PWR061
 U 1 1 5817A25E
 P 1300 2100
-F 0 "#PWR53" H 1300 1850 50  0001 C CNN
+F 0 "#PWR061" H 1300 1850 50  0001 C CNN
 F 1 "GNDA" H 1305 1927 50  0000 C CNN
 F 2 "" H 1300 2100 50  0000 C CNN
@@
 NoConn ~ 6750 3500
 $Comp
-L +3.3VP #PWR64
+L +3.3VP #PWR062
 U 1 1 5817DDD0
 P 5550 4400
-F 0 "#PWR64" H 5700 4350 50  0001 C CNN
+F 0 "#PWR062" H 5700 4350 50  0001 C CNN
 F 1 "+3.3VP" V 5570 4498 50  0000 L CNN
 F 2 "" H 5550 4400 50  0000 C CNN
@@
 $EndComp
 $Comp
-L +3.3VP #PWR61
+L +3.3VP #PWR063
 U 1 1 5817DF9D
 P 3600 5500
-F 0 "#PWR61" H 3750 5450 50  0001 C CNN
+F 0 "#PWR063" H 3750 5450 50  0001 C CNN
 F 1 "+3.3VP" H 3620 5643 50  0000 C CNN
 F 2 "" H 3600 5500 50  0000 C CNN
@@
 $EndComp
 $Comp
-L +3.3VP #PWR56
+L +3.3VP #PWR064
 U 1 1 5817E8B4
 P 2300 5500
-F 0 "#PWR56" H 2450 5450 50  0001 C CNN
+F 0 "#PWR064" H 2450 5450 50  0001 C CNN
 F 1 "+3.3VP" H 2320 5643 50  0000 C CNN
 F 2 "" H 2300 5500 50  0000 C CNN
@@
 $EndComp
 $Comp
-L +3.3VP #PWR70
+L +3.3VP #PWR065
 U 1 1 5817F6CE
 P 10075 3975
-F 0 "#PWR70" H 10225 3925 50  0001 C CNN
+F 0 "#PWR065" H 10225 3925 50  0001 C CNN
 F 1 "+3.3VP" H 10095 4118 50  0000 C CNN
 F 2 "" H 10075 3975 50  0000 C CNN
@@
 $EndComp
 $Comp
-L +3.3VP #PWR52
+L +3.3VP #PWR066
 U 1 1 581811E3
 P 875 2475
-F 0 "#PWR52" H 1025 2425 50  0001 C CNN
+F 0 "#PWR066" H 1025 2425 50  0001 C CNN
 F 1 "+3.3VP" H 895 2618 50  0000 C CNN
 F 2 "" H 875 2475 50  0000 C CNN
@@
 $EndComp
 $Comp
-L +3.3VP #PWR54
+L +3.3VP #PWR067
 U 1 1 58182A98
 P 1650 2475
-F 0 "#PWR54" H 1800 2425 50  0001 C CNN
+F 0 "#PWR067" H 1800 2425 50  0001 C CNN
 F 1 "+3.3VP" H 1670 2618 50  0000 C CNN
 F 2 "" H 1650 2475 50  0000 C CNN
@@
 $EndComp
 $Comp
-L +3.3VP #PWR58
+L +3.3VP #PWR068
 U 1 1 58182C81
 P 2425 2475
-F 0 "#PWR58" H 2575 2425 50  0001 C CNN
+F 0 "#PWR068" H 2575 2425 50  0001 C CNN
 F 1 "+3.3VP" H 2445 2618 50  0000 C CNN
 F 2 "" H 2425 2475 50  0000 C CNN
@@
 $EndComp
 $Comp
-L +3.3VP #PWR60
+L +3.3VP #PWR069
 U 1 1 58183424
 P 3200 2475
-F 0 "#PWR60" H 3350 2425 50  0001 C CNN
+F 0 "#PWR069" H 3350 2425 50  0001 C CNN
 F 1 "+3.3VP" H 3220 2618 50  0000 C CNN
 F 2 "" H 3200 2475 50  0000 C CNN
@@
 $EndComp
 $Comp
-L VAA #PWR66
+L VAA #PWR070
 U 1 1 58184D5C
-P 6025 3500
-F 0 "#PWR66" H 6025 3350 50  0001 C CNN
-F 1 "VAA" V 6043 3627 50  0000 L CNN
-F 2 "" H 6025 3500 50  0000 C CNN
-F 3 "" H 6025 3500 50  0000 C CNN
-	1    6025 3500
+P 6025 4300
+F 0 "#PWR070" H 6025 4150 50  0001 C CNN
+F 1 "VAA" V 6043 4427 50  0000 L CNN
+F 2 "" H 6025 4300 50  0000 C CNN
+F 3 "" H 6025 4300 50  0000 C CNN
+	1    6025 4300
 	0    -1   -1   0
 $EndComp
 $Comp
-L VAA #PWR68
+L VAA #PWR071
 U 1 1 58185AC0
 P 9550 1400
-F 0 "#PWR68" H 9550 1250 50  0001 C CNN
+F 0 "#PWR071" H 9550 1250 50  0001 C CNN
 F 1 "VAA" H 9567 1573 50  0000 C CNN
 F 2 "" H 9550 1400 50  0000 C CNN
@@
 	1    0    0    -1
 $EndComp
+Wire Wire Line
+	6025 4300 6125 4300
+NoConn ~ 6125 3500
 $EndSCHEMATC
