File: hw-design/bluetooth.sch (KiCad schematic (older format))
At the start: 22 parts, among them U7 BlueNRG, U8 BALF-NRG-01D3, Y2 32kHz, Y3 16MHz

Commit message: PCB 1.2 almost done, only shape could be improved.
Parts:
- L1, L2: footprint w_smd_inductors:inductor_smd_0603 -> w_smd_cap:c_0603
Changed lines of the file:
@@
 F 0 "L1" V 8241 4550 50  0000 C CNN
 F 1 "INDUCTOR" V 8150 4550 50  0000 C CNN
-F 2 "w_smd_inductors:inductor_smd_0603" H 8025 4550 50  0001 C CNN
+F 2 "w_smd_cap:c_0603" H 8025 4550 50  0001 C CNN
 F 3 "" H 8025 4550 50  0000 C CNN
 	1    8025 4550
@@
 F 0 "L2" V 8291 3250 50  0000 C CNN
 F 1 "3.9 nH" V 8200 3250 50  0000 C CNN
-F 2 "w_smd_inductors:inductor_smd_0603" H 8075 3250 50  0001 C CNN
+F 2 "w_smd_cap:c_0603" H 8075 3250 50  0001 C CNN
 F 3 "" H 8075 3250 50  0000 C CNN
 	1    8075 3250
